File: KiCad/Fuimini-V2.kicad_sch (KiCad schematic)
At the start: 59 parts, among them SW1 1TS026A-1100-0550-CT, T1 MHPA0808RGBDT, U1 ANT162442ST-1000AM1, U2 NRF52833-QDAA-R, U3 ICM-45686, U4 IST8306, U5 SSP7615-33DFR, U6 LGS4056HDA, U7 EA8103, X1 XL4EL89CKI-111YLC-32M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

Commit message: - Moved IMU decoupling caps closer to IMU - Updated IMU footprint - Smoothed 2.4GHz RF trace - Disconnected 2.4GHz RF reference gnd from main gnd plane - Connected nRF pin 37 (gnd) to center ground pad - Added second 10uF output capacitor to DCDC, measured to reduce ripple   by 4mV
Parts:
- added C1n5: 10uF, beaLib:C_0402_JLC, symbol Device:C_Small
Connections:
- net GND: now also C1n5.1
- net VDD nRF: now also C1n5.2
Changed lines of the file:
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@@
 	)
 	(junction
+		(at 100.33 128.27)
+		(diameter 0)
+		(color 0 0 0 0)
+	)
+	(junction
 		(at 152.4 82.55)
 		(diameter 0)
@@
 	)
 	(junction
+		(at 100.33 123.19)
+		(diameter 0)
+		(color 0 0 0 0)
+	)
+	(junction
 		(at 116.84 146.05)
 		(diameter 0)
@@
 	(wire
 		(pts
+			(xy 96.52 128.27) (xy 100.33 128.27)
+		)
+		(stroke
+			(width 0)
+			(type default)
+		)
+	)
+	(wire
+		(pts
 			(xy 67.31 118.11) (xy 67.31 120.65)
 		)
@@
 		)
 	)
+	(wire
+		(pts
+			(xy 96.52 123.19) (xy 100.33 123.19)
+		)
+		(stroke
+			(width 0)
+			(type default)
+		)
+	)
 	(global_label "DCEN"
 		(shape input)
@@
 		(dnp no)
 		(property "Reference" "C1n2"
-			(at 144.272 126.492 0)
+			(at 144.78 126.746 0)
 			(effects
 				(font
@@
 		)
 		(property "Value" "10uF"
-			(at 144.018 124.46 0)
+			(at 144.526 124.714 0)
 			(effects
 				(font
@@
 		(dnp no)
 		(property "Reference" "C1n3"
-			(at 98.298 124.968 0)
+			(at 98.806 130.048 0)
 			(effects
 				(font
@@
 		)
 		(property "Value" "10uF"
-			(at 98.552 127 0)
+			(at 99.06 132.08 0)
 			(effects
 				(font
@@
 					(unit 1)
 				)
+			)
+		)
+	)
+	(symbol
+		(lib_id "Device:C_Small")
+		(at 96.52 125.73 180)
+		(unit 1)
+		(exclude_from_sim no)
+		(in_bom yes)
+		(on_board yes)
+		(dnp no)
+		(property "Reference" "C1n5"
+			(at 99.06 134.112 0)
+			(effects
+				(font
+					(size 1.27 1.27)
+				)
+				(justify left)
+			)
+		)
+		(property "Value" "10uF"
+			(at 99.314 136.144 0)
+			(effects
+				(font
+					(size 1.27 1.27)
+				)
+				(justify left)
+			)
+		)
+		(property "Footprint" "beaLib:C_0402_JLC"
+			(at 96.52 125.73 0)
+			(effects
+				(font
+					(size 1.27 1.27)
+				)
+				(hide yes)
+			)
+		)
+		(property "Datasheet" "~"
+			(at 96.52 125.73 0)
+			(effects
+				(font
+					(size 1.27 1.27)
+				)
+				(hide yes)
+			)
+		)
+		(property "Description" "Unpolarized capacitor, small symbol"
+			(at 96.52 125.73 0)
+			(effects
+				(font
+					(size 1.27 1.27)
+				)
+				(hide yes)
+			)
+		)
+		(pin "1"
+		)
+		(pin "2"
+		)
+		(instances
+			(project "Fuimini-V2"
+				(path "/7f675c71-ed66-43d9-81bf-09a8e18818c7"
+					(reference "C1n5")
+					(unit 1)
+				)
