File: KiCad/Fuimini-V2.kicad_pcb (KiCad board)
At the start: 4 copper layers, 15 x 29.2 mm, 60 parts, among them SW1 1TS026A-1100-0550-CT, T1 MHPA0808RGBDT, U1 ANT162442ST-1000AM1, U2 NRF52833-QDAA-R, U3 ICM-45686, U4 IST8306, U5 SSP7615-33DFR, U6 LGS4056HDA, U7 EA8103, X1 XL4EL89CKI-111YLC-32M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

Commit message: - Added test points for VBUS and VDD
Parts:
- added REF**: TestPoint_Pad_D1.0mm, TestPoint:TestPoint_Pad_D1.0mm, B.Cu at (106.7, 94.2)
- added REF**: TestPoint_Pad_D1.0mm, TestPoint:TestPoint_Pad_D1.0mm, B.Cu at (105.3, 92.0)
Routing:
- net VDD nRF: track 83.1 -> 86.0 mm
- net VBUS: track 37.4 -> 39.2 mm
Other:
- board text added: "1.8"
- board text added: "5"
- board text added: "Added VBUS test point -"
- board text added: "Added VDD test point -"
- board text removed: "* changed layer stackup, In1.Cu now ground plane."
- board text removed: "- Added mag footprint"
- board text removed: "- Moved trace to go around clock, rather than directly beneath it"
- board text removed: "- added missing vias to radiator - added missing bottom layer to radiator - changed radiator width from 0.6 to 0.5mm"
- board text removed: "- changed frequency tuning capacitor value & DNP'd one"
- board text removed: "- extended ground plane up"
- board text removed: "- fixed ground short on RF transmission line"
- board text removed: "- fixed misshapen top ground plane on RF transmission line"
- board text removed: "- fixed missing bottom ground plane on RF transmission line"
- board text removed: "- fixed pin 7,10,11 being tied to GND (causes current draw)"
- board text removed: "- moved switch ~0.25mm inward (was sticking out too much)"

Commit message: - Moved IMU decoupling caps closer to IMU - Updated IMU footprint - Smoothed 2.4GHz RF trace - Disconnected 2.4GHz RF reference gnd from main gnd plane - Connected nRF pin 37 (gnd) to center ground pad - Added second 10uF output capacitor to DCDC, measured to reduce ripple   by 4mV
Parts:
- removed the REF** at (106.7, 94.2)
- added C1n5: 10uF, beaLib:C_0402_JLC, F.Cu at (115.3, 107.3)
- U3: footprint imu_custom:ICM-42688-P -> imu_custom:IMU
- moved C2i1 1.07 mm to (106.4, 93.1), turned to -90 degrees
- moved X2 0.17 mm to (104.5, 92.6)
Routing:
- net VDD nRF: track 86.0 -> 81.0 mm, vias 10 -> 11
- net GND: track 80.7 -> 85.0 mm, vias 45 -> 50
- net CLK: track 2.01 -> 2.96 mm
- net Net-(U7-SWITCH): track 0.99 -> 0.05 mm
- net CLK_EN: track 11.6 -> 12.4 mm
- net VBUS: track 39.2 -> 40.0 mm
Other:
- board text added: "- Added second 10uF output capacitor to DCDC This was measured to reduce voltage ripple by ~4mV"
- board text added: "- Connected GND pin to pad"
- board text added: "Disconnected RF ref. gnd from main gnd-"
- board text added: "MPS5.1.2"
- board text added: "Moved IMU decoupling caps closer -"
- board text added: "Smoothed RF trace-"
- board text added: "Updated IMU footprint, now using meia's -"
- board text removed: "1.8"
- board text removed: "5"
- board text removed: "Added VDD test point -"
- board text removed: "MPS5.1.1"

Commit message: - Updated PCB dont remember what (￣y▽,￣)╭ - Updated case design dont remember what (/▽＼)
Parts:
- L1, L2: footprint Inductor_SMD:L_0201_0603Metric -> easyeda2kicad:L0201-RD
- moved R1 0.43 mm to (108.3, 91.8), turned to -90 degrees
- moved R2C3 0.19 mm to (117.0, 100.1)
- moved C1 0.13 mm to (111.4, 106.6)
- moved C3r1 0.13 mm to (116.0, 92.8)
- moved C1i1 0.11 mm to (108.5, 92.9)
- moved R2C2 0.11 mm to (115.7, 99.4)
- moved C1n1 0.11 mm to (105.0, 104.6)
- moved R1R2 0.09 mm to (113.1, 109.2)
- moved R2D2 0.08 mm to (113.2, 107.7)
- moved C1n3 0.07 mm to (114.4, 107.2)
- moved L2 0.05 mm to (107.6, 106.1)
- moved C14 0.05 mm to (103.6, 111.0)
- moved R1D2 0.05 mm to (113.2, 106.5)
Routing:
- net VDD nRF: track 81.0 -> 78.6 mm
- net GND: track 85.0 -> 84.4 mm
Other:
- board text added: "- Updated C_0201 footprints to match JLC's - Updated R_0201 footprints to match JLC's - Adjusted some spacings to better match new footprints - Added solder mask expansions to footprints (values from JLC)"
- board text added: "MPS5.2.0"
- board text added: "Shortened path from 1v8 via to imu -"
- board text removed: "MPS5.1.2"
